Commit message: change cube's dynamics and mass

File: helping_hands_rl_envs/pybullet/urdf/object/cube.urdf (robot description, URDF)
Before this commit: robot cube, 1 links, 0 joints
Links:
- link baseLink: mass 0.1 -> 0.8

Commit message: Merge branch 'beta' of github.com:SaulBatman/helping_hands_rl_envs into beta

File: helping_hands_rl_envs/pybullet/urdf/object/cube.urdf (robot description, URDF)
Before this commit: robot cube, 1 links, 0 joints
Links:
- link baseLink: mass 0.8 -> 0.1
